File: Power Supply/PCB/KiCad files/RTSS_Power_Supply_V2-5C.kicad_sch (KiCad schematic)
At the start: 68 parts, among them J1 Barrel_Jack, J2 Ext LED, J4 Conn_01x01, J5 SMA_connector, J6 5V fan, J7 12V fan, Q1 IRF640N, SW1 SW_SPST, U1 L7812, U2 L7805, U3 74LVC1GU04, U4 74LVC1G14, U5 74HC161, U6 1EDN8511B, Y1 7.6MHz

Commit message: Update PCB to V2.5C
Changed reference designators for continuity and updated Digikey BOMs
Parts:
- renumbered C22 to C10, C11 to C101, C12 to C102, C13 to C103, C14 to C104, C15 to C105, C16 to C106, C17 to C107, C18 to C108, C19 to C109, C24 to C11, C20 to C110, C21 to C111, C10 to C12, C7 to C3, C3 to C4, C4 to C5, C5 to C6, C6 to C7, J5 to J101, J6 to J2, J7 to J3, J2 to J4, J4 to J5, L1 to L101, L2 to L102, L3 to L103, L4 to L104, L5 to L105, Q1 to Q101, R4 to R101, R5 to R102, R6 to R103, R7 to R104, R9 to R2, R8 to R3, R2 to R4, R3 to R5, TP5 to TP101, TP6 to TP102, TP7 to TP103, TP8 to TP104, TP9 to TP105, TP10 to TP106
Other:
- note added: "All capacitors in the RF section should be rated for at least 200V and be Class I (i.e. C0G/NP0). Inductors L102-L105 should be wound on Kool Mu 0077932A7 cores using 22AWG or larger magnet wire. Approximate number of inductor turns: L102 = 14, L103 = 23, L104 = 23, L105 = 19 Measure inductances at 475kHz on a VNA or at least 100kHz on a LCR. Try to be within ±0.2uH. When tuning the inductors, ma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"
- note removed: "All capacitors in the RF section should be rated for at least 200V and be Class I (i.e. C0G/NP0). Inductors L2-L5 should be wound on Kool Mu 0077932A7 cores using 22AWG or larger magnet wire. Approximate number of inductor turns: L2 = 14, L3 = 23, L4 = 23, L5 = 19 Measure inductances at 475kHz on a VNA or at least 100kHz on a LCR. Try to be within ±0.2uH. When tuning the inductors, make the coils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"
